File: ts_23_LV_BMS_MASTER/LV_MASTER_A_SAMPLE/LV_MASTER_A_SAMPLE.kicad_pcb (KiCad board)
At the start: 4 copper layers, 77.5 x 46.9 mm, 117 parts, among them J1 DT 12P, J2 UART, J3 BOOT1, J4 STLINK, J5 Conn_01x02_Male, J6 Conn_02x02_Counter_Clockwise, J7 Conn_02x02_Counter_Clockwise, Q1 STD7NK40Z, Q2 STD7NK40Z, T1 HX1188NL, U1 STM32F446RET7, U2 TLV70033_SOT23-5, U4 ADM3053, U5 B82786C0104H002, U6 LTC6820, U7 ISO1540, U8 ADS1115, U9 ADUM3221, Y1 ECS-80-18-30-JGN-TR, Y2 FC-135_32.7680KA-A5

Commit message: LV_BMS PCB Uploads
Other:
- board text added: "0.3364 mm"
- board text added: "1.2000 mm"
- board text added: "7. Surface finish: OSP"
- board text added: "9. Total Thickness: 1.2mm"
- board text added: "OSP"
- board text removed: "0.469733 mm"
- board text removed: "1.6000 mm"
- board text removed: "7. Surface finish: HASL (Lead Free)"
- board text removed: "9. Total Thickness: 1.6mm"
- board text removed: "HAL lead-free"
